File: Ver 0.0 Rel 0.1/PCB & schematic/Visually impaired v6 panel - v1.sch (EAGLE design)
At the start: 146 parts, among them J10 DF11-8DP-2DSA, J11 BM02B-SRSS-TB, J2 DF11-8DP-2DSA, J3 DF11-8DP-2DSA, J4 BM02B-SRSS-TB, J5 DF11-8DP-2DSA, M1 2RB18Z1BS, M2 2RB18Z1BS, P1 CB-AA-PC-POS, P2 CB-AA-PC-NEG, Q1 DMG1023UV, Q2 DMG1023UV, Q3 2N7002, T1 TCT40-16T, T2 TCT40-16T, U1 MCP1700T-3002E/TT, U10 74LVC08A, U11 TC7SB3157CFU, U12 LMV324IPWR, U13 S25FL127SABMFI101, U14 23LC512-I/ST, U15 PAM8404KG, U16 AK4386ET, U17 FXOS8700CQR1, U18 SE97BTP, U19 AT24C02, U2 MKL16Z256VLH4, U20 TMP101, U3 AAT3693, U4 MCP1640T-I/CHY, U5 NLAS4157, U6 AAT2120, U7 NLAS4157, U8 NLAS4157, U9 NLAS4157, Y1 9HT7-32.768KDZF-T

Commit message: Components consolidation & OM
Parts:
- C12, C13: PARTNO STOCK: DK 587-1227-1-ND -> DK: 490-6349-1-ND
- C17: PARTNO STOCK: DK 587-1227-1-ND -> DK: 490-1312-1-ND
- C37: PARTNO DK: 490-10432-1-ND -> DK: 490-10435-1-ND
- C48, C49, C50: PARTNO * -> STOCK: DK 587-1227-1-ND
- C51: PARTNO * -> DK: 490-1312-1-ND
- C8: PARTNO STOCK: DK 311-1459-1-ND -> DK: 490-10470-1-ND
- L7: PARTNO * -> DK: 553-2374-1-ND
- R18: PARTNO DK:RC0603FR-0775KL -> DK: 311-22.0KLRCT-ND
- R2: PARTNO * -> DK: 311-10.0KLRCT-ND
- R22: PARTNO DK: 311-10.0KLRCT-ND -> DK: 1276-4063-1-ND
